File: six_month/Arduino_Nano.kicad_sch (KiCad schematic)
At the start: 3 parts, among them J3 Conn_01x15, J5 Conn_01x15

Commit message: Changes
Removed the microphone idea, added a DAC for Bluetooth to Line out. Allows for external speakers to be connected via an Aux cable
Other:
- note added: "NANO ESP32"
- moved on the sheet: A1, J3, J5
