File: six_month/DAC.kicad_sch (KiCad schematic)
At the start: 0 parts

Commit message: Added Audio Connector
Included 3.5mm TRS for External Speakers from the DAC.
Parts:
- added C10, C14, C5, C8: 0.1u, symbol Device:C
- added C11, C12: 2.2u, symbol Device:C
- added C13, C6, C7, C9: 10u, symbol Device:C_Polarized
- added C15, C16: 2.2n, symbol Device:C
- added J1: PJ313D, syms_foots:AUDIO-TH_PJ313D, symbol syms_foots:PJ313D
- added R11, R12: 470, symbol Device:R_US
- added U6: PCM5102APWR, syms_foots:TSSOP-20_L6.5-W4.4-P0.65-LS6.4-BL, symbol syms_foots:PCM5102APWR
Connections:
- new net: C10.1, C9.1, U6.1 (CPVDD)
- new net: C5.1, C6.1, U6.18 (LDOO)
- new net: C11.2, U6.2 (CAPP)
- new net: C11.1, U6.4 (CAPM)
- new net: C12.1, U6.5 (VNEG)
- new net: R12.1, U6.6 (OUTL)
- new net: R11.1, U6.7 (OUTR)
- new net: C15.1, R12.2
- new net +3V3_VCC: C7.1, C8.1, U6.20 (DVDD)
- new net GND: C10.2, C12.2, C13.2, C14.2, C15.2, C16.2, C5.2, C6.2, C7.2, C8.2, C9.2, J1.2, U6.10 (DEMP), U6.11 (FLT), U6.12 (SCK), U6.16 (FMT), U6.19 (DGND), U6.3 (CPGND), U6.9 (AGND)
- new net I2S_CLK: U6.13 (BCK)
- new net I2S_DIN: U6.14 (DIN)
- new net I2S_WS: U6.15 (LRCK)
- new net L_CH: C13.1, C14.1, J1.3, U6.8 (AVDD)
- new net R_CH: C16.1, J1.4, R11.2
- no-connect marks 0 -> 1
Other:
- note added: "DAC and Aux Output"
