File: six_month/Display.kicad_sch (KiCad schematic)
At the start: 0 parts

Commit message: Removed some stuff
Removed the speaker stuff because we dont need it.
Other:
- note added: "using this display https://www.adafruit.com/product/4741#technical-details"
Changed lines of the file:
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@@
 	(generator_version "9.0")
 	(paper "A4")
+	(text "using this display https://www.adafruit.com/product/4741#technical-details"
+		(exclude_from_sim no)
+		(at 136.144 75.946 0)
+		(effects
+			(font
+				(size 1.27 1.27)
+			)
+		)
+	)
 )
