File: six_month/temp.kicad_sch (KiCad schematic)
At the start: 5 parts, among them U4 BME688_C3664478

Commit message: Changes
Removed the microphone idea, added a DAC for Bluetooth to Line out. Allows for external speakers to be connected via an Aux cable
Changed lines of the file:
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@@
 		)
 	)
-	(text_box "I2C Address: 1110110 (0x76)"
+	(text_box "I2C Address: 0x76"
 		(exclude_from_sim no)
 		(at 33.274 26.162 0)
@@
 			)
 		)
-		(property "Datasheet" ""
+		(property "Datasheet" "https://www.bosch-sensortec.com/products/environmental-sensors/gas-sensors/bme688/"
 			(at 66.04 54.61 0)
 			(effects

Commit message: Added Audio Connector
Included 3.5mm TRS for External Speakers from the DAC.
Other:
- note added: "Temp/Humidity Sensor"
- moved on the sheet: C1, C2, D2, D3, U4
